Commit message: Finished parameterized kicking solver

File: motion_planning/nao.urdf (robot description, URDF)
Before this commit: robot naoH25V40, 43 links, 42 joints
Links:
- removed link LFinger11_link
- removed link LFinger12_link
- removed link LFinger13_link
- removed link LFinger21_link
- removed link LFinger22_link
- removed link LFinger23_link
- removed link LThumb1_link
- removed link LThumb2_link
- removed link RFinger11_link
- removed link RFinger12_link
- removed link RFinger13_link
- removed link RFinger21_link
- removed link RFinger22_link
- removed link RFinger23_link
- removed link RThumb1_link
- removed link RThumb2_link
Joints:
- removed joint LFinger11
- removed joint LFinger12
- removed joint LFinger13
- removed joint LFinger21
- removed joint LFinger22
- removed joint LFinger23
- removed joint LThumb1
- removed joint LThumb2
- removed joint RFinger11
- removed joint RFinger12
- removed joint RFinger13
- removed joint RFinger21
- removed joint RFinger22
- removed joint RFinger23
- removed joint RThumb1
- removed joint RThumb2
- joint HeadPitch: limit lower=-0.671952 upper=0.514872 effort=1.532 velocity=7.19407 -> lower=-0.671952 upper=0.514872 effort=1.532 velocity=1.0
- joint HeadYaw: limit lower=-2.08567 upper=2.08567 effort=1.547 velocity=8.26797 -> lower=-2.08567 upper=2.08567 effort=1.547 velocity=1.0
- joint LAnklePitch: limit lower=-1.18944 upper=0.922581 effort=3.023 velocity=6.40239 -> lower=-1.18944 upper=0.922581 effort=3.023 velocity=1.0
- joint LAnkleRoll: limit lower=-0.397761 upper=0.768992 effort=3.348 velocity=4.16174 -> lower=-0.397761 upper=0.768992 effort=3.348 velocity=1.0
- joint LElbowRoll: limit lower=-1.54462 upper=-0.0349066 effort=1.532 velocity=7.19407 -> lower=-1.54462 upper=-0.0349066 effort=1.532 velocity=1.0
- joint LElbowYaw: limit lower=-2.08567 upper=2.08567 effort=1.547 velocity=8.26797 -> lower=-2.08567 upper=2.08567 effort=1.547 velocity=1.0
- joint LHand: limit lower=0 upper=1.0 effort=0.292 velocity=8.33 -> lower=0 upper=1.0 effort=0.292 velocity=1.0
- joint LHipPitch: limit lower=-1.53589 upper=0.48398 effort=3.023 velocity=6.40239 -> lower=-1.53589 upper=0.48398 effort=3.023 velocity=1.0
- joint LHipRoll: limit lower=-0.379435 upper=0.79046 effort=3.348 velocity=4.16174 -> lower=-0.379435 upper=0.79046 effort=3.348 velocity=1.0
- joint LHipYawPitch: limit lower=-1.14529 upper=0.740718 effort=3.348 velocity=4.16174 -> lower=-1.14529 upper=0.740718 effort=3.348 velocity=1.0
- joint LKneePitch: limit lower=-0.0923279 upper=2.11255 effort=3.023 velocity=6.40239 -> lower=-0.0923279 upper=2.11255 effort=3.023 velocity=1.0
- joint LShoulderPitch: limit lower=-2.08567 upper=2.08567 effort=1.329 velocity=8.26797 -> lower=0 upper=1.4 effort=1.329 velocity=1.0
- joint LShoulderRoll: limit lower=-0.314159 upper=1.32645 effort=1.7835 velocity=7.19407 -> lower=0 upper=1.32645 effort=1.7835 velocity=1.0
- joint LWristYaw: limit lower=-1.82387 upper=1.82387 effort=0.4075 velocity=24.6229 -> lower=-1.82387 upper=1.82387 effort=0.4075 velocity=1.0
- joint RAnklePitch: limit lower=-1.1863 upper=0.932006 effort=3.0226 velocity=6.40239 -> lower=-1.1863 upper=0.932006 effort=3.0226 velocity=1.0
- joint RAnkleRoll: limit lower=-0.768992 upper=0.397761 effort=3.348 velocity=4.16174 -> lower=-0.768992 upper=0.397761 effort=3.348 velocity=1.0
- joint RElbowRoll: limit lower=0.0349066 upper=1.54462 effort=1.532 velocity=7.19407 -> lower=0.0349066 upper=1.54462 effort=1.532 velocity=1.0
- joint RElbowYaw: limit lower=-2.08567 upper=2.08567 effort=1.547 velocity=8.26797 -> lower=-2.08567 upper=2.08567 effort=1.547 velocity=1.0
- joint RHand: limit lower=0 upper=1.0 effort=0.292 velocity=8.33 -> lower=0 upper=1.0 effort=0.292 velocity=1.0
- joint RHipPitch: limit lower=-1.53589 upper=0.48398 effort=3.0226 velocity=6.40239 -> lower=-1.53589 upper=0.48398 effort=3.0226 velocity=1.0
- joint RHipRoll: limit lower=-0.79046 upper=0.379435 effort=3.348 velocity=4.16174 -> lower=-0.79046 upper=0.379435 effort=3.348 velocity=1.0
- joint RHipYawPitch: limit lower=-1.14529 upper=0.740718 effort=3.348 velocity=4.16174 -> lower=-1.14529 upper=0.740718 effort=3.348 velocity=1.0
- joint RKneePitch: limit lower=-0.0923279 upper=2.11255 effort=3.0226 velocity=6.40239 -> lower=-0.0923279 upper=2.11255 effort=3.0226 velocity=1.0
- joint RShoulderPitch: limit lower=-2.08567 upper=2.08567 effort=1.329 velocity=8.26797 -> lower=0 upper=1.4 effort=1.329 velocity=1.0
- joint RShoulderRoll: limit lower=-1.32645 upper=0.314159 effort=1.783 velocity=7.19407 -> lower=-1.32645 upper=0 effort=1.783 velocity=1.0
- joint RWristYaw: limit lower=-1.82387 upper=1.82387 effort=0.4075 velocity=24.6229 -> lower=-1.82387 upper=1.82387 effort=0.4075 velocity=1.0

Commit message: Improved joint name ordering, increased movement speed

File: motion_planning/nao.urdf (robot description, URDF)
Before this commit: robot naoH25V40, 27 links, 26 joints
Joints:
- joint HeadPitch: limit lower=-0.671952 upper=0.514872 effort=1.532 velocity=1.0 -> lower=-0.671952 upper=0.514872 effort=1.532 velocity=1.25
- joint HeadYaw: limit lower=-2.08567 upper=2.08567 effort=1.547 velocity=1.0 -> lower=-2.08567 upper=2.08567 effort=1.547 velocity=1.25
- joint LAnklePitch: limit lower=-1.18944 upper=0.922581 effort=3.023 velocity=1.0 -> lower=-1.18944 upper=0.922581 effort=3.023 velocity=1.75
- joint LAnkleRoll: limit lower=-0.397761 upper=0.768992 effort=3.348 velocity=1.0 -> lower=-0.397761 upper=0.768992 effort=3.348 velocity=1.75
- joint LElbowRoll: limit lower=-1.54462 upper=-0.0349066 effort=1.532 velocity=1.0 -> lower=-1.54462 upper=-0.0349066 effort=1.532 velocity=0.1
- joint LElbowYaw: limit lower=-2.08567 upper=2.08567 effort=1.547 velocity=1.0 -> lower=-2.08567 upper=2.08567 effort=1.547 velocity=0.1
- joint LHand: limit lower=0 upper=1.0 effort=0.292 velocity=1.0 -> lower=0 upper=1.0 effort=0.292 velocity=1.25
- joint LHipPitch: limit lower=-1.53589 upper=0.48398 effort=3.023 velocity=1.0 -> lower=-1.53589 upper=0.48398 effort=3.023 velocity=1.75
- joint LHipRoll: limit lower=-0.379435 upper=0.79046 effort=3.348 velocity=1.0 -> lower=-0.379435 upper=0.79046 effort=3.348 velocity=1.75
- joint LHipYawPitch: limit lower=-1.14529 upper=0.740718 effort=3.348 velocity=1.0 -> lower=-1.14529 upper=0.740718 effort=3.348 velocity=1.75
- joint LKneePitch: limit lower=-0.0923279 upper=2.11255 effort=3.023 velocity=1.0 -> lower=-0.0923279 upper=2.11255 effort=3.023 velocity=1.75
- joint LShoulderPitch: limit lower=0 upper=1.4 effort=1.329 velocity=1.0 -> lower=0 upper=1.4 effort=1.329 velocity=1.25
- joint LShoulderRoll: limit lower=0 upper=1.32645 effort=1.7835 velocity=1.0 -> lower=0 upper=1.32645 effort=1.7835 velocity=1.25
- joint LWristYaw: limit lower=-1.82387 upper=1.82387 effort=0.4075 velocity=1.0 -> lower=-1.82387 upper=1.82387 effort=0.4075 velocity=1.25
- joint RAnklePitch: limit lower=-1.1863 upper=0.932006 effort=3.0226 velocity=1.0 -> lower=-1.1863 upper=0.932006 effort=3.0226 velocity=1.75
- joint RAnkleRoll: limit lower=-0.768992 upper=0.397761 effort=3.348 velocity=1.0 -> lower=-0.768992 upper=0.397761 effort=3.348 velocity=1.75
- joint RElbowRoll: limit lower=0.0349066 upper=1.54462 effort=1.532 velocity=1.0 -> lower=0.0349066 upper=1.54462 effort=1.532 velocity=0.1
- joint RElbowYaw: limit lower=-2.08567 upper=2.08567 effort=1.547 velocity=1.0 -> lower=-2.08567 upper=2.08567 effort=1.547 velocity=0.1
- joint RHand: limit lower=0 upper=1.0 effort=0.292 velocity=1.0 -> lower=0 upper=1.0 effort=0.292 velocity=1.25
- joint RHipPitch: limit lower=-1.53589 upper=0.48398 effort=3.0226 velocity=1.0 -> lower=-1.53589 upper=0.48398 effort=3.0226 velocity=1.75
- joint RHipRoll: limit lower=-0.79046 upper=0.379435 effort=3.348 velocity=1.0 -> lower=-0.79046 upper=0.379435 effort=3.348 velocity=1.75
- joint RHipYawPitch: limit lower=-1.14529 upper=0.740718 effort=3.348 velocity=1.0 -> lower=-1.14529 upper=0.740718 effort=3.348 velocity=1.75
- joint RKneePitch: limit lower=-0.0923279 upper=2.11255 effort=3.0226 velocity=1.0 -> lower=-0.0923279 upper=2.11255 effort=3.0226 velocity=1.75
- joint RShoulderPitch: limit lower=0 upper=1.4 effort=1.329 velocity=1.0 -> lower=0 upper=1.4 effort=1.329 velocity=1.25
- joint RShoulderRoll: limit lower=-1.32645 upper=0 effort=1.783 velocity=1.0 -> lower=-1.32645 upper=0 effort=1.783 velocity=1.25
- joint RWristYaw: limit lower=-1.82387 upper=1.82387 effort=0.4075 velocity=1.0 -> lower=-1.82387 upper=1.82387 effort=0.4075 velocity=1.25

Commit message: More kick tweaks

File: motion_planning/nao.urdf (robot description, URDF)
Before this commit: robot naoH25V40, 27 links, 26 joints
Joints:
- joint LShoulderRoll: limit lower=0 upper=1.32645 effort=1.7835 velocity=1.25 -> lower=0.3 upper=1.32645 effort=1.7835 velocity=1.25
- joint RShoulderRoll: limit lower=-1.32645 upper=0 effort=1.783 velocity=1.25 -> lower=-1.32645 upper=-0.3 effort=1.783 velocity=1.25

Commit message: Updated sparse kick

File: motion_planning/nao.urdf (robot description, URDF)
Before this commit: robot naoH25V40, 27 links, 26 joints
Joints:
- joint LElbowRoll: limit lower=-1.54462 upper=-0.0349066 effort=1.532 velocity=0.1 -> lower=0 upper=0 effort=1.532 velocity=0.1
- joint LElbowYaw: limit lower=-2.08567 upper=2.08567 effort=1.547 velocity=0.1 -> lower=0 upper=0 effort=1.547 velocity=0.1
- joint LHand: limit lower=0 upper=1.0 effort=0.292 velocity=1.25 -> lower=0 upper=0 effort=0.292 velocity=1.25
- joint LWristYaw: limit lower=-1.82387 upper=1.82387 effort=0.4075 velocity=1.25 -> lower=-0 upper=0 effort=0.4075 velocity=1.25
- joint RElbowRoll: limit lower=0.0349066 upper=1.54462 effort=1.532 velocity=0.1 -> lower=0 upper=0 effort=1.532 velocity=0.1
- joint RElbowYaw: limit lower=-2.08567 upper=2.08567 effort=1.547 velocity=0.1 -> lower=0 upper=0 effort=1.547 velocity=0.1
- joint RHand: limit lower=0 upper=1.0 effort=0.292 velocity=1.25 -> lower=0 upper=0 effort=0.292 velocity=1.25
- joint RWristYaw: limit lower=-1.82387 upper=1.82387 effort=0.4075 velocity=1.25 -> lower=0 upper=0 effort=0.4075 velocity=1.25

Commit message: Updated sparse kick

File: motion_planning/nao.urdf (robot description, URDF)
Before this commit: robot naoH25V40, 27 links, 26 joints
Joints:
- joint LElbowRoll: limit lower=0 upper=0 effort=1.532 velocity=0.1 -> lower=-1.54462 upper=-0.0349066 effort=1.532 velocity=0.1
- joint LElbowYaw: limit lower=0 upper=0 effort=1.547 velocity=0.1 -> lower=-2.08567 upper=2.08567 effort=1.547 velocity=0.1
- joint LHand: limit lower=0 upper=0 effort=0.292 velocity=1.25 -> lower=0 upper=1.0 effort=0.292 velocity=1.25
- joint LWristYaw: limit lower=-0 upper=0 effort=0.4075 velocity=1.25 -> lower=-1.82387 upper=1.82387 effort=0.4075 velocity=1.25
- joint RElbowRoll: limit lower=0 upper=0 effort=1.532 velocity=0.1 -> lower=0.0349066 upper=1.54462 effort=1.532 velocity=0.1
- joint RElbowYaw: limit lower=0 upper=0 effort=1.547 velocity=0.1 -> lower=-2.08567 upper=2.08567 effort=1.547 velocity=0.1
- joint RHand: limit lower=0 upper=0 effort=0.292 velocity=1.25 -> lower=0 upper=1.0 effort=0.292 velocity=1.25
- joint RWristYaw: limit lower=0 upper=0 effort=0.4075 velocity=1.25 -> lower=-1.82387 upper=1.82387 effort=0.4075 velocity=1.25

Commit message: Added a hopefully improved online balancer

File: motion_planning/nao.urdf (robot description, URDF)
Before this commit: robot naoH25V40, 27 links, 26 joints
Links:
- added link l_sole
- added link r_sole
Joints:
- added joint LLeg_effector_fixedjoint: type fixed, parent l_ankle, child l_sole, origin xyz=0 0 -0.04511 rpy=0 0 0, axis 0 0 0
- added joint RLeg_effector_fixedjoint: type fixed, parent r_ankle, child r_sole, origin xyz=0 0 -0.04511 rpy=0 0 0, axis 0 0 0

Commit message: Fixed arm issue

File: motion_planning/nao.urdf (robot description, URDF)
Before this commit: robot naoH25V40, 29 links, 28 joints
Joints:
- joint LShoulderPitch: limit lower=0 upper=1.4 effort=1.329 velocity=1.25 -> lower=1.5 upper=1.6 effort=1.329 velocity=1.25
- joint RShoulderPitch: limit lower=0 upper=1.4 effort=1.329 velocity=1.25 -> lower=1.5 upper=1.6 effort=1.329 velocity=1.25

Commit message: Added goal space weighting, CoM z regulation

File: motion_planning/nao.urdf (robot description, URDF)
Before this commit: robot naoH25V40, 29 links, 28 joints
Joints:
- joint LKneePitch: limit lower=-0.0923279 upper=2.11255 effort=3.023 velocity=1.75 -> lower=0.01 upper=2.11255 effort=3.023 velocity=1.75
- joint RKneePitch: limit lower=-0.0923279 upper=2.11255 effort=3.0226 velocity=1.75 -> lower=0.01 upper=2.11255 effort=3.0226 velocity=1.75

Commit message: Added support knee straightener

File: motion_planning/nao.urdf (robot description, URDF)
Before this commit: robot naoH25V40, 29 links, 28 joints
Joints:
- joint LKneePitch: limit lower=0.01 upper=2.11255 effort=3.023 velocity=1.75 -> lower=0.05 upper=1.57 effort=3.023 velocity=1.75
- joint RKneePitch: limit lower=0.01 upper=2.11255 effort=3.0226 velocity=1.75 -> lower=0.05 upper=1.57 effort=3.0226 velocity=1.75
